Commit message: poc: multi-board working

File: description/ros2_control/inmoov_ros2_control.xacro (robot description, xacro)
@@ -14,38 +14,230 @@
       </xacro:unless>
     </hardware>
-      <joint name="left_shoulder_z_joint">
+      <joint name="i02_leftHand_ThumbMid_joint">
           <param name="virtual_pin">0</param>
           <param name="servo_type">180</param>
-          <param name="offset">1.5708</param>
-          <param name="direction">1</param>
-          <param name="scale">1</param>
-          <param name="limit_min">0</param>
-          <param name="limit_max">3.14159</param>
-          <param name="default">1.5708</param>
-          <command_interface name="torque_enable"/>
-          <command_interface name="position">
-            <param name="min">-0.872665</param>
-            <param name="max">0.610865</param>
-          </command_interface>
-          <state_interface name="position" />
-      </joint>
-      <joint name="left_shoulder_x_joint">
+          <param name="offset">0</param>
+          <param name="direction">1</param>
+          <param name="scale">0.84082</param>
+          <param name="limit_min">0</param>
+          <param name="limit_max">1.39626</param>
+          <param name="default">0</param>
+          <command_interface name="torque_enable"/>
+          <command_interface name="position">
+            <param name="min">0.0</param>
+            <param name="max">1.174</param>
+          </command_interface>
+          <state_interface name="position" />
+      </joint>
+      <joint name="i02_leftHand_indexPhal_joint">
           <param name="virtual_pin">1</param>
           <param name="servo_type">180</param>
           <param name="offset">0</param>
           <param name="direction">1</param>
-          <param name="scale">1</param>
-          <param name="limit_min">0</param>
-          <param name="limit_max">3.14159</param>
-          <param name="default">0</param>
-          <command_interface name="torque_enable"/>
-          <command_interface name="position">
-            <param name="min">-0.349066</param>
+          <param name="scale">0.57384</param>
+          <param name="limit_min">0</param>
+          <param name="limit_max">2.26893</param>
+          <param name="default">0</param>
+          <command_interface name="torque_enable"/>
+          <command_interface name="position">
+            <param name="min">0.0</param>
+            <param name="max">1.302</param>
+          </command_interface>
+          <state_interface name="position" />
+      </joint>
+      <joint name="i02_leftHand_majeurePhal_joint">
+          <param name="virtual_pin">2</param>
+          <param name="servo_type">180</param>
+          <param name="offset">0</param>
+          <param name="direction">1</param>
+          <param name="scale">0.55533</param>
+          <param name="limit_min">0</param>
+          <param name="limit_max">2.26893</param>
+          <param name="default">0</param>
+          <command_interface name="torque_enable"/>
+          <command_interface name="position">
+            <param name="min">0.0</param>
+            <param name="max">1.26</param>
+          </command_interface>
+          <state_interface name="position" />
+      </joint>
+      <joint name="i02_leftHand_ringFingerPhal_joint">
+          <param name="virtual_pin">3</param>
+          <param name="servo_type">180</param>
+          <param name="offset">0</param>
+          <param name="direction">1</param>
+          <param name="scale">0.60513</param>
+          <param name="limit_min">0</param>
+          <param name="limit_max">2.26893</param>
+          <param name="default">0</param>
+          <command_interface name="torque_enable"/>
+          <command_interface name="position">
+            <param name="min">0.0</param>
+            <param name="max">1.373</param>
+          </command_interface>
+          <state_interface name="position" />
+      </joint>
+      <joint name="i02_leftHand_pinkyPhal_joint">
+          <param name="virtual_pin">4</param>
+          <param name="servo_type">180</param>
+          <param name="offset">2.96706</param>
+          <param name="direction">-1</param>
+          <param name="scale">0.45769</param>
+          <param name="limit_min">0</param>
+          <param name="limit_max">2.96706</param>
+          <param name="default">2.96706</param>
+          <command_interface name="torque_enable"/>
+          <command_interface name="position">
+            <param name="min">0.0</param>
+            <param name="max">1.358</param>
+          </command_interface>
+          <state_interface name="position" />
+      </joint>
+      <joint name="left_wrist_z_joint">
+          <param name="virtual_pin">5</param>
+          <param name="servo_type">180</param>
+          <param name="offset">2.61799</param>
+          <param name="direction">1</param>
+          <param name="scale">1</param>
+          <param name="limit_min">0</param>
+          <param name="limit_max">3.14159</param>
+          <param name="default">2.61799</param>
+          <command_interface name="torque_enable"/>
+          <command_interface name="position">
+            <param name="min">-1.570796</param>
+            <param name="max">1.570796</param>
+          </command_interface>
+          <state_interface name="position" />
+      </joint>
+      <joint name="i02_rightHand_ThumbMid_joint">
+          <param name="virtual_pin">6</param>
+          <param name="servo_type">180</param>
+          <param name="offset">0</param>
+          <param name="direction">1</param>
+          <param name="scale">0.82291</param>
+          <param name="limit_min">0</param>
+          <param name="limit_max">1.39626</param>
+          <param name="default">0</param>
+          <command_interface name="torque_enable"/>
+          <command_interface name="position">
+            <param name="min">0.0</param>
+            <param name="max">1.149</param>
+          </command_interface>
+          <state_interface name="position" />
+      </joint>
+      <joint name="i02_rightHand_indexPhal_joint">
+          <param name="virtual_pin">7</param>
+          <param name="servo_type">180</param>
+          <param name="offset">0</param>
+          <param name="direction">1</param>
+          <param name="scale">0.55885</param>
+          <param name="limit_min">0</param>
+          <param name="limit_max">2.26893</param>
+          <param name="default">0</param>
+          <command_interface name="torque_enable"/>
+          <command_interface name="position">
+            <param name="min">0.0</param>
+            <param name="max">1.268</param>
+          </command_interface>
+          <state_interface name="position" />
+      </joint>
+      <joint name="i02_rightHand_majeurePhal_joint">
+          <param name="virtual_pin">8</param>
+          <param name="servo_type">180</param>
+          <param name="offset">0</param>
+          <param name="direction">1</param>
+          <param name="scale">0.41317</param>
+          <param name="limit_min">0</param>
+          <param name="limit_max">3.14159</param>
+          <param name="default">0</param>
+          <command_interface name="torque_enable"/>
+          <command_interface name="position">
+            <param name="min">0.0</param>
+            <param name="max">1.298</param>
+          </command_interface>
+          <state_interface name="position" />
+      </joint>
+      <joint name="i02_rightHand_ringFingerPhal_joint">
+          <param name="virtual_pin">9</param>
+          <param name="servo_type">180</param>
+          <param name="offset">0</param>
+          <param name="direction">1</param>
+          <param name="scale">0.58001</param>
+          <param name="limit_min">0</param>
+          <param name="limit_max">2.26893</param>
+          <param name="default">0</param>
+          <command_interface name="torque_enable"/>
+          <command_interface name="position">
+            <param name="min">0.0</param>
+            <param name="max">1.316</param>
+          </command_interface>
+          <state_interface name="position" />
+      </joint>
+      <joint name="i02_rightHand_pinkyPhal_joint">
+          <param name="virtual_pin">10</param>
+          <param name="servo_type">180</param>
+          <param name="offset">0</param>
+          <param name="direction">1</param>
+          <param name="scale">0.57208</param>
+          <param name="limit_min">0</param>
+          <param name="limit_max">2.26893</param>
+          <param name="default">0</param>
+          <command_interface name="torque_enable"/>
+          <command_interface name="position">
+            <param name="min">0.0</param>
+            <param name="max">1.298</param>
+          </command_interface>
+          <state_interface name="position" />
+      </joint>
+      <joint name="right_wrist_z_joint">
+          <param name="virtual_pin">11</param>
+          <param name="servo_type">180</param>
+          <param name="offset">2.61799</param>
+          <param name="direction">-1</param>
+          <param name="scale">1</param>
+          <param name="limit_min">0</param>
+          <param name="limit_max">3.14159</param>
+          <param name="default">2.61799</param>
+          <command_interface name="torque_enable"/>
+          <command_interface name="position">
+            <param name="min">-1.570796</param>
+            <param name="max">1.570796</param>
+          </command_interface>
+          <state_interface name="position" />
+      </joint>
+      <joint name="right_shoulder_z_joint">
+          <param name="virtual_pin">12</param>
+          <param name="servo_type">180</param>
+          <param name="offset">1.5708</param>
+          <param name="direction">-1</param>
+          <param name="scale">1</param>
+          <param name="limit_min">0</param>
+          <param name="limit_max">3.14159</param>
+          <param name="default">1.5708</param>
+          <command_interface name="torque_enable"/>
+          <command_interface name="position">
+            <param name="min">-0.610865</param>
+            <param name="max">0.837758</param>
+          </command_interface>
+          <state_interface name="position" />
+      </joint>
+      <joint name="right_shoulder_x_joint">
+          <param name="virtual_pin">13</param>
+          <param name="servo_type">180</param>
+          <param name="offset">0</param>
+          <param name="direction">1</param>
+          <param name="scale">1</param>
+          <param name="limit_min">0</param>
+          <param name="limit_max">3.14159</param>
+          <param name="default">0</param>
+          <command_interface name="torque_enable"/>
+          <command_interface name="position">
+            <param name="min">-0.523599</param>
             <param name="max">2.356194</param>
           </command_interface>
           <state_interface name="position" />
       </joint>
-      <joint name="left_elbow_x_joint">
-          <param name="virtual_pin">2</param>
+      <joint name="right_elbow_x_joint">
+          <param name="virtual_pin">14</param>
           <param name="servo_type">180</param>
           <param name="offset">0</param>
@@ -62,86 +254,38 @@
           <state_interface name="position" />
       </joint>
-      <joint name="left_shoulder_y_joint">
-          <param name="virtual_pin">3</param>
-          <param name="servo_type">180</param>
-          <param name="offset">0</param>
-          <param name="direction">1</param>
-          <param name="scale">1</param>
-          <param name="limit_min">0</param>
-          <param name="limit_max">3.14159</param>
-          <param name="default">0</param>
-          <command_interface name="torque_enable"/>
-          <command_interface name="position">
-            <param name="min">0.0</param>
-            <param name="max">1.134464</param>
-          </command_interface>
-          <state_interface name="position" />
-      </joint>
-      <joint name="i01_head_rothead_joint">
-          <param name="virtual_pin">4</param>
-          <param name="servo_type">180</param>
-          <param name="offset">1.5708</param>
-          <param name="direction">1</param>
-          <param name="scale">1</param>
-          <param name="limit_min">0</param>
-          <param name="limit_max">3.14159</param>
-          <param name="default">1.5708</param>
-          <command_interface name="torque_enable"/>
-          <command_interface name="position">
-            <param name="min">-1.047198</param>
-            <param name="max">0.872665</param>
-          </command_interface>
-          <state_interface name="position" />
-      </joint>
-      <joint name="neck_joint">
-          <param name="virtual_pin">5</param>
-          <param name="servo_type">180</param>
-          <param name="offset">1.5708</param>
-          <param name="direction">1</param>
-          <param name="scale">1</param>
-          <param name="limit_min">0</param>
-          <param name="limit_max">3.14159</param>
-          <param name="default">1.5708</param>
-          <command_interface name="torque_enable"/>
-          <command_interface name="position">
-            <param name="min">-0.349066</param>
-            <param name="max">0.349066</param>
-          </command_interface>
-          <state_interface name="position" />
-      </joint>
-      <joint name="i01_head_neck_001_joint">
-          <param name="virtual_pin">6</param>
-          <param name="servo_type">180</param>
-          <param name="offset">1.5708</param>
-          <param name="direction">1</param>
-          <param name="scale">1</param>
-          <param name="limit_min">0</param>
-          <param name="limit_max">3.14159</param>
-          <param name="default">1.5708</param>
-          <command_interface name="torque_enable"/>
-          <command_interface name="position">
-            <param name="min">-0.349066</param>
-            <param name="max">0.349066</param>
-          </command_interface>
-          <state_interface name="position" />
-      </joint>
-      <joint name="i02_head_jaw_joint">
-          <param name="virtual_pin">7</param>
-          <param name="servo_type">180</param>
-          <param name="offset">0.43633</param>
-          <param name="direction">1</param>
-          <param name="scale">0.10526</param>
-          <param name="limit_min">0.43633</param>
-          <param name="limit_max">2.0944</param>
-          <param name="default">0.43633</param>
-          <command_interface name="torque_enable"/>
-          <command_interface name="position">
-            <param name="min">0.0</param>
-            <param name="max">0.17453</param>
-          </command_interface>
-          <state_interface name="position" />
-      </joint>
-      <joint name="i02_head_right_eye_vertical_joint">
-          <param name="virtual_pin">8</param>
+      <joint name="right_shoulder_y_joint">
+          <param name="virtual_pin">15</param>
+          <param name="servo_type">180</param>
+          <param name="offset">0</param>
+          <param name="direction">1</param>
+          <param name="scale">1</param>
+          <param name="limit_min">0</param>
+          <param name="limit_max">3.14159</param>
+          <param name="default">0</param>
+          <command_interface name="torque_enable"/>
+          <command_interface name="position">
+            <param name="min">0.0</param>
+            <param name="max">1.22173</param>
+          </command_interface>
+          <state_interface name="position" />
+      </joint>
+      <joint name="torso_z_joint">
+          <param name="virtual_pin">16</param>
+          <param name="servo_type">180</param>
+          <param name="offset">2.35619</param>
+          <param name="direction">1</param>
+          <param name="scale">1</param>
+          <param name="limit_min">0</param>
+          <param name="limit_max">3.14159</param>
+          <param name="default">2.35619</param>
+          <command_interface name="torque_enable"/>
+          <command_interface name="position">
+            <param name="min">-0.523599</param>
+            <param name="max">0.523599</param>
+          </command_interface>
+          <state_interface name="position" />
+      </joint>
+      <joint name="torso_y_joint">
+          <param name="virtual_pin">17</param>
           <param name="servo_type">180</param>
           <param name="offset">1.5708</param>
@@ -155,52 +299,4 @@
             <param name="min">-0.261799</param>
             <param name="max">0.261799</param>
-          </command_interface>
-          <state_interface name="position" />
-      </joint>
-      <joint name="i02_head_right_eye_horizontal_joint">
-          <param name="virtual_pin">9</param>
-          <param name="servo_type">180</param>
-          <param name="offset">1.5708</param>
-          <param name="direction">1</param>
-          <param name="scale">1</param>
-          <param name="limit_min">0</param>
-          <param name="limit_max">3.14159</param>
-          <param name="default">1.5708</param>
-          <command_interface name="torque_enable"/>
-          <command_interface name="position">
-            <param name="min">-0.174533</param>
-            <param name="max">0.174533</param>
-          </command_interface>
-          <state_interface name="position" />
-      </joint>
-      <joint name="i02_head_left_eye_vertical_joint">
-          <param name="virtual_pin">10</param>
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