Commit message: docs: launch the i2 with robot_package and describe its model_scale

File: description/robot_description/urdf/properties.xacro (robot description, xacro)
@@ -1,13 +1,12 @@
 <?xml version="1.0"?>
 <!--
-LinkForge (Blender) exports inmoov_i2.urdf.xacro in raw CAD/Blender scene
-units, not meters — every <origin xyz> and <mesh scale> in that file is
-written as ${model_scale*...} against this property.
+LinkForge (Blender) exports robot_description.urdf.xacro in raw CAD/Blender
+scene units, not meters: every joint, visual and collision <origin xyz> and
+<mesh scale> in that file is written as ${model_scale*...} against this property.
 0.10604 (2026-10-05) is recalibrated against the physical robot: in the zero
 pose the crown is 1.81 m above the floor, stand included. It replaced 0.1196,
-carried over from the old Sentience-Robotics inmoov_urdf properties.xacro.
-The mass/inertia estimate (scripts/inertia_estimate.json) is stored in SI
-units for this scale: after changing model_scale, recompute it with
-scripts/claude_compute_inertia.py and re-apply it.
+carried over from the inmoov_urdf properties.xacro.
+The inertials are in SI units for this scale: re-estimate them after changing
+model_scale.
 -->
 <robot xmlns:xacro="http://www.ros.org/wiki/xacro">
