Commit message: feat(hardware): drive the i2 from two Arduino Megas

File: description/gazebo/gazebo.xacro (robot description, xacro)
@@ -2,5 +2,5 @@
 <!-- Generated by lucy_config_generator - do not edit. -->
 <robot xmlns:xacro="http://www.ros.org/wiki/xacro" name="inmoov" version="1.0">
-  <ros2_control name="LucyHardwareLeftArm" type="system">
+  <ros2_control name="LucyHardwareArms" type="system">
     <hardware>
       <plugin>gz_ros2_control/GazeboSimSystem</plugin>
@@ -8,5 +8,5 @@
     <joint name="left_shoulder_z_joint">
       <param name="virtual_pin">0</param>
-      <param name="servo_type">270</param>
+      <param name="servo_type">180</param>
       <param name="offset">1.5708</param>
       <param name="direction">1</param>
@@ -20,5 +20,5 @@
     <joint name="left_shoulder_x_joint">
       <param name="virtual_pin">1</param>
-      <param name="servo_type">270</param>
+      <param name="servo_type">180</param>
       <param name="offset">0</param>
       <param name="direction">1</param>
@@ -32,5 +32,5 @@
     <joint name="left_elbow_x_joint">
       <param name="virtual_pin">2</param>
-      <param name="servo_type">270</param>
+      <param name="servo_type">180</param>
       <param name="offset">0</param>
       <param name="direction">1</param>
@@ -44,10 +44,10 @@
     <joint name="left_wrist_z_joint">
       <param name="virtual_pin">3</param>
-      <param name="servo_type">300</param>
+      <param name="servo_type">180</param>
       <param name="offset">2.61799</param>
       <param name="direction">1</param>
       <param name="scale">1</param>
       <param name="limit_min">0</param>
-      <param name="limit_max">5.23599</param>
+      <param name="limit_max">3.14159</param>
       <param name="default">2.61799</param>
       <command_interface name="position" />
@@ -56,5 +56,5 @@
     <joint name="i02_leftHand_ThumbMid_joint">
       <param name="virtual_pin">4</param>
-      <param name="servo_type">300</param>
+      <param name="servo_type">180</param>
       <param name="offset">0</param>
       <param name="direction">1</param>
@@ -68,5 +68,5 @@
     <joint name="i02_leftHand_indexPhal_joint">
       <param name="virtual_pin">5</param>
-      <param name="servo_type">300</param>
+      <param name="servo_type">180</param>
       <param name="offset">0</param>
       <param name="direction">1</param>
@@ -80,5 +80,5 @@
     <joint name="i02_leftHand_majeurePhal_joint">
       <param name="virtual_pin">6</param>
-      <param name="servo_type">300</param>
+      <param name="servo_type">180</param>
       <param name="offset">0</param>
       <param name="direction">1</param>
@@ -92,5 +92,5 @@
     <joint name="i02_leftHand_ringFingerPhal_joint">
       <param name="virtual_pin">7</param>
-      <param name="servo_type">300</param>
+      <param name="servo_type">180</param>
       <param name="offset">0</param>
       <param name="direction">1</param>
@@ -104,22 +104,17 @@
     <joint name="i02_leftHand_pinkyPhal_joint">
       <param name="virtual_pin">8</param>
-      <param name="servo_type">300</param>
-      <param name="offset">0</param>
-      <param name="direction">1</param>
-      <param name="scale">1</param>
-      <param name="limit_min">0</param>
-      <param name="limit_max">3.14159</param>
-      <param name="default">0</param>
-      <command_interface name="position" />
-      <state_interface name="position" />
-    </joint>
-  </ros2_control>
-  <ros2_control name="LucyHardwareRightArm" type="system">
-    <hardware>
-      <plugin>gz_ros2_control/GazeboSimSystem</plugin>
-    </hardware>
+      <param name="servo_type">180</param>
+      <param name="offset">0</param>
+      <param name="direction">1</param>
+      <param name="scale">1</param>
+      <param name="limit_min">0</param>
+      <param name="limit_max">3.14159</param>
+      <param name="default">0</param>
+      <command_interface name="position" />
+      <state_interface name="position" />
+    </joint>
     <joint name="right_shoulder_z_joint">
-      <param name="virtual_pin">0</param>
-      <param name="servo_type">270</param>
+      <param name="virtual_pin">9</param>
+      <param name="servo_type">180</param>
       <param name="offset">1.5708</param>
       <param name="direction">-1</param>
@@ -132,6 +127,6 @@
     </joint>
     <joint name="right_shoulder_x_joint">
-      <param name="virtual_pin">1</param>
-      <param name="servo_type">270</param>
+      <param name="virtual_pin">10</param>
+      <param name="servo_type">180</param>
       <param name="offset">0</param>
       <param name="direction">1</param>
@@ -144,6 +139,6 @@
     </joint>
     <joint name="right_elbow_x_joint">
-      <param name="virtual_pin">2</param>
-      <param name="servo_type">270</param>
+      <param name="virtual_pin">11</param>
+      <param name="servo_type">180</param>
       <param name="offset">0</param>
       <param name="direction">1</param>
@@ -156,11 +151,11 @@
     </joint>
     <joint name="right_wrist_z_joint">
-      <param name="virtual_pin">3</param>
-      <param name="servo_type">300</param>
+      <param name="virtual_pin">12</param>
+      <param name="servo_type">180</param>
       <param name="offset">2.61799</param>
       <param name="direction">-1</param>
       <param name="scale">1</param>
       <param name="limit_min">0</param>
-      <param name="limit_max">5.23599</param>
+      <param name="limit_max">3.14159</param>
       <param name="default">2.61799</param>
       <command_interface name="position" />
@@ -168,6 +163,6 @@
     </joint>
     <joint name="i02_rightHand_ThumbMid_joint">
-      <param name="virtual_pin">4</param>
-      <param name="servo_type">300</param>
+      <param name="virtual_pin">13</param>
+      <param name="servo_type">180</param>
       <param name="offset">0</param>
       <param name="direction">1</param>
@@ -180,6 +175,6 @@
     </joint>
     <joint name="i02_rightHand_indexPhal_joint">
-      <param name="virtual_pin">5</param>
-      <param name="servo_type">300</param>
+      <param name="virtual_pin">14</param>
+      <param name="servo_type">180</param>
       <param name="offset">0</param>
       <param name="direction">1</param>
@@ -192,6 +187,6 @@
     </joint>
     <joint name="i02_rightHand_majeurePhal_joint">
-      <param name="virtual_pin">6</param>
-      <param name="servo_type">300</param>
+      <param name="virtual_pin">15</param>
+      <param name="servo_type">180</param>
       <param name="offset">0</param>
       <param name="direction">1</param>
@@ -204,6 +199,6 @@
     </joint>
     <joint name="i02_rightHand_ringFingerPhal_joint">
-      <param name="virtual_pin">7</param>
-      <param name="servo_type">300</param>
+      <param name="virtual_pin">16</param>
+      <param name="servo_type">180</param>
       <param name="offset">0</param>
       <param name="direction">1</param>
@@ -216,6 +211,6 @@
     </joint>
     <joint name="i02_rightHand_pinkyPhal_joint">
-      <param name="virtual_pin">8</param>
-      <param name="servo_type">300</param>
+      <param name="virtual_pin">17</param>
+      <param name="servo_type">180</param>
       <param name="offset">0</param>
       <param name="direction">1</param>
@@ -234,5 +229,5 @@
     <joint name="left_shoulder_y_joint">
       <param name="virtual_pin">0</param>
-      <param name="servo_type">270</param>
+      <param name="servo_type">180</param>
       <param name="offset">0</param>
       <param name="direction">1</param>
@@ -246,5 +241,5 @@
     <joint name="right_shoulder_y_joint">
       <param name="virtual_pin">1</param>
-      <param name="servo_type">270</param>
+      <param name="servo_type">180</param>
       <param name="offset">0</param>
       <param name="direction">1</param>
@@ -258,10 +253,10 @@
     <joint name="torso_z_joint">
       <param name="virtual_pin">2</param>
-      <param name="servo_type">270</param>
+      <param name="servo_type">180</param>
       <param name="offset">2.35619</param>
       <param name="direction">1</param>
       <param name="scale">1</param>
       <param name="limit_min">0</param>
-      <param name="limit_max">4.71239</param>
+      <param name="limit_max">3.14159</param>
       <param name="default">2.35619</param>
       <command_interface name="position" />
@@ -270,5 +265,5 @@
     <joint name="torso_y_joint">
       <param name="virtual_pin">3</param>
-      <param name="servo_type">270</param>
+      <param name="servo_type">180</param>
       <param name="offset">1.5708</param>
       <param name="direction">1</param>
@@ -282,5 +277,5 @@
     <joint name="i01_head_rothead_joint">
       <param name="virtual_pin">4</param>
-      <param name="servo_type">270</param>
+      <param name="servo_type">180</param>
       <param name="offset">1.5708</param>
       <param name="direction">1</param>
@@ -294,5 +289,5 @@
     <joint name="neck_joint">
       <param name="virtual_pin">5</param>
-      <param name="servo_type">270</param>
+      <param name="servo_type">180</param>
       <param name="offset">1.5708</param>
       <param name="direction">1</param>
@@ -306,5 +301,5 @@
     <joint name="i01_head_neck_001_joint">
       <param name="virtual_pin">6</param>
-      <param name="servo_type">300</param>
+      <param name="servo_type">180</param>
       <param name="offset">1.5708</param>
       <param name="direction">1</param>
@@ -318,5 +313,5 @@
     <joint name="i02_head_jaw_joint">
       <param name="virtual_pin">7</param>
-      <param name="servo_type">300</param>
+      <param name="servo_type">180</param>
       <param name="offset">0.43633</param>
       <param name="direction">1</param>

File: description/ros2_control/inmoov_ros2_control.xacro (robot description, xacro)
@@ -3,5 +3,5 @@
 <robot xmlns:xacro="http://www.ros.org/wiki/xacro" name="inmoov" version="1.0">
   <xacro:arg name="use_mock_hardware" default="false" />
-  <ros2_control name="LucyHardwareLeftArm" type="system">
+  <ros2_control name="LucyHardwareArms" type="system">
     <hardware>
       <plugin>lucy_ros2_control/LucySystemHardware</plugin>
@@ -10,11 +10,11 @@
       </xacro:if>
       <xacro:unless value="$(arg use_mock_hardware)">
-        <param name="publisher_topic">actuators/left_arm</param>
-        <param name="node_name">left_arm</param>
+        <param name="publisher_topic">actuators/arms</param>
+        <param name="node_name">arms</param>
       </xacro:unless>
     </hardware>
       <joint name="left_shoulder_z_joint">
           <param name="virtual_pin">0</param>
-          <param name="servo_type">270</param>
+          <param name="servo_type">180</param>
           <param name="offset">1.5708</param>
           <param name="direction">1</param>
@@ -32,5 +32,5 @@
       <joint name="left_shoulder_x_joint">
           <param name="virtual_pin">1</param>
-          <param name="servo_type">270</param>
+          <param name="servo_type">180</param>
           <param name="offset">0</param>
           <param name="direction">1</param>
@@ -48,5 +48,5 @@
       <joint name="left_elbow_x_joint">
           <param name="virtual_pin">2</param>
-          <param name="servo_type">270</param>
+          <param name="servo_type">180</param>
           <param name="offset">0</param>
           <param name="direction">1</param>
@@ -64,10 +64,10 @@
       <joint name="left_wrist_z_joint">
           <param name="virtual_pin">3</param>
-          <param name="servo_type">300</param>
+          <param name="servo_type">180</param>
           <param name="offset">2.61799</param>
           <param name="direction">1</param>
           <param name="scale">1</param>
           <param name="limit_min">0</param>
-          <param name="limit_max">5.23599</param>
+          <param name="limit_max">3.14159</param>
           <param name="default">2.61799</param>
           <command_interface name="torque_enable"/>
@@ -80,5 +80,5 @@
       <joint name="i02_leftHand_ThumbMid_joint">
           <param name="virtual_pin">4</param>
-          <param name="servo_type">300</param>
+          <param name="servo_type">180</param>
           <param name="offset">0</param>
           <param name="direction">1</param>
@@ -96,5 +96,5 @@
       <joint name="i02_leftHand_indexPhal_joint">
           <param name="virtual_pin">5</param>
-          <param name="servo_type">300</param>
+          <param name="servo_type">180</param>
           <param name="offset">0</param>
           <param name="direction">1</param>
@@ -112,5 +112,5 @@
       <joint name="i02_leftHand_majeurePhal_joint">
           <param name="virtual_pin">6</param>
-          <param name="servo_type">300</param>
+          <param name="servo_type">180</param>
           <param name="offset">0</param>
           <param name="direction">1</param>
@@ -128,5 +128,5 @@
       <joint name="i02_leftHand_ringFingerPhal_joint">
           <param name="virtual_pin">7</param>
-          <param name="servo_type">300</param>
+          <param name="servo_type">180</param>
           <param name="offset">0</param>
           <param name="direction">1</param>
@@ -144,5 +144,5 @@
       <joint name="i02_leftHand_pinkyPhal_joint">
           <param name="virtual_pin">8</param>
-          <param name="servo_type">300</param>
+          <param name="servo_type">180</param>
           <param name="offset">0</param>
           <param name="direction">1</param>
@@ -158,19 +158,7 @@
           <state_interface name="position" />
       </joint>
-  </ros2_control>
-  <ros2_control name="LucyHardwareRightArm" type="system">
-    <hardware>
-      <plugin>lucy_ros2_control/LucySystemHardware</plugin>
-      <xacro:if value="$(arg use_mock_hardware)">
-        <param name="publish_actuators">false</param>
-      </xacro:if>
-      <xacro:unless value="$(arg use_mock_hardware)">
-        <param name="publisher_topic">actuators/right_arm</param>
-        <param name="node_name">right_arm</param>
-      </xacro:unless>
-    </hardware>
       <joint name="right_shoulder_z_joint">
-          <param name="virtual_pin">0</param>
-          <param name="servo_type">270</param>
+          <param name="virtual_pin">9</param>
+          <param name="servo_type">180</param>
           <param name="offset">1.5708</param>
           <param name="direction">-1</param>
@@ -187,6 +175,6 @@
       </joint>
       <joint name="right_shoulder_x_joint">
-          <param name="virtual_pin">1</param>
-          <param name="servo_type">270</param>
+          <param name="virtual_pin">10</param>
+          <param name="servo_type">180</param>
           <param name="offset">0</param>
           <param name="direction">1</param>
@@ -203,6 +191,6 @@
       </joint>
       <joint name="right_elbow_x_joint">
-          <param name="virtual_pin">2</param>
-          <param name="servo_type">270</param>
+          <param name="virtual_pin">11</param>
+          <param name="servo_type">180</param>
           <param name="offset">0</param>
           <param name="direction">1</param>
@@ -219,11 +207,11 @@
       </joint>
       <joint name="right_wrist_z_joint">
-          <param name="virtual_pin">3</param>
-          <param name="servo_type">300</param>
+          <param name="virtual_pin">12</param>
+          <param name="servo_type">180</param>
           <param name="offset">2.61799</param>
           <param name="direction">-1</param>
           <param name="scale">1</param>
           <param name="limit_min">0</param>
-          <param name="limit_max">5.23599</param>
+          <param name="limit_max">3.14159</param>
           <param name="default">2.61799</param>
           <command_interface name="torque_enable"/>
@@ -235,6 +223,6 @@
       </joint>
       <joint name="i02_rightHand_ThumbMid_joint">
-          <param name="virtual_pin">4</param>
-          <param name="servo_type">300</param>
+          <param name="virtual_pin">13</param>
+          <param name="servo_type">180</param>
           <param name="offset">0</param>
           <param name="direction">1</param>
@@ -251,6 +239,6 @@
       </joint>
       <joint name="i02_rightHand_indexPhal_joint">
-          <param name="virtual_pin">5</param>
-          <param name="servo_type">300</param>
+          <param name="virtual_pin">14</param>
+          <param name="servo_type">180</param>
           <param name="offset">0</param>
           <param name="direction">1</param>
@@ -267,6 +255,6 @@
       </joint>
       <joint name="i02_rightHand_majeurePhal_joint">
-          <param name="virtual_pin">6</param>
-          <param name="servo_type">300</param>
+          <param name="virtual_pin">15</param>
+          <param name="servo_type">180</param>
           <param name="offset">0</param>
           <param name="direction">1</param>
@@ -283,6 +271,6 @@
       </joint>
       <joint name="i02_rightHand_ringFingerPhal_joint">
-          <param name="virtual_pin">7</param>
-          <param name="servo_type">300</param>
+          <param name="virtual_pin">16</param>
+          <param name="servo_type">180</param>
           <param name="offset">0</param>
           <param name="direction">1</param>
@@ -299,6 +287,6 @@
       </joint>
       <joint name="i02_rightHand_pinkyPhal_joint">
-          <param name="virtual_pin">8</param>
-          <param name="servo_type">300</param>
+          <param name="virtual_pin">17</param>
+          <param name="servo_type">180</param>
           <param name="offset">0</param>
           <param name="direction">1</param>
@@ -328,5 +316,5 @@
       <joint name="left_shoulder_y_joint">
           <param name="virtual_pin">0</param>
-          <param name="servo_type">270</param>
+          <param name="servo_type">180</param>
           <param name="offset">0</param>
           <param name="direction">1</param>
@@ -344,5 +332,5 @@
       <joint name="right_shoulder_y_joint">
           <param name="virtual_pin">1</param>
-          <param name="servo_type">270</param>
+          <param name="servo_type">180</param>
           <param name="offset">0</param>
           <param name="direction">1</param>
@@ -360,10 +348,10 @@
       <joint name="torso_z_joint">
           <param name="virtual_pin">2</param>
-          <param name="servo_type">270</param>
+          <param name="servo_type">180</param>
           <param name="offset">2.35619</param>
           <param name="direction">1</param>
           <param name="scale">1</param>
           <param name="limit_min">0</param>
-          <param name="limit_max">4.71239</param>
+          <param name="limit_max">3.14159</param>
           <param name="default">2.35619</param>
           <command_interface name="torque_enable"/>
@@ -376,5 +364,5 @@
       <joint name="torso_y_joint">
           <param name="virtual_pin">3</param>
-          <param name="servo_type">270</param>
+          <param name="servo_type">180</param>
           <param name="offset">1.5708</param>
           <param name="direction">1</param>
@@ -392,5 +380,5 @@
       <joint name="i01_head_rothead_joint">
           <param name="virtual_pin">4</param>
-          <param name="servo_type">270</param>
+          <param name="servo_type">180</param>
           <param name="offset">1.5708</param>
           <param name="direction">1</param>
@@ -408,5 +396,5 @@
       <joint name="neck_joint">
           <param name="virtual_pin">5</param>
-          <param name="servo_type">270</param>
+          <param name="servo_type">180</param>
           <param name="offset">1.5708</param>
           <param name="direction">1</param>
@@ -424,5 +412,5 @@
       <joint name="i01_head_neck_001_joint">
           <param name="virtual_pin">6</param>
-          <param name="servo_type">300</param>
+          <param name="servo_type">180</param>
           <param name="offset">1.5708</param>
           <param name="direction">1</param>
@@ -440,5 +428,5 @@
       <joint name="i02_head_jaw_joint">
           <param name="virtual_pin">7</param>
-          <param name="servo_type">300</param>
+          <param name="servo_type">180</param>
           <param name="offset">0.43633</param>
           <param name="direction">1</param>
