Commit message: feat(hardware): mega_left / mega_right layout and PoC_InMoovI2

File: description/gazebo/gazebo.xacro (robot description, xacro)
@@ -2,5 +2,5 @@
 <!-- Generated by lucy_config_generator - do not edit. -->
 <robot xmlns:xacro="http://www.ros.org/wiki/xacro" name="inmoov" version="1.0">
-  <ros2_control name="LucyHardwareArms" type="system">
+  <ros2_control name="LucyHardwareLeft" type="system">
     <hardware>
       <plugin>gz_ros2_control/GazeboSimSystem</plugin>
@@ -42,234 +42,13 @@
       <state_interface name="position" />
     </joint>
-    <joint name="left_wrist_z_joint">
+    <joint name="left_shoulder_y_joint">
       <param name="virtual_pin">3</param>
       <param name="servo_type">180</param>
-      <param name="offset">2.61799</param>
-      <param name="direction">1</param>
-      <param name="scale">1</param>
-      <param name="limit_min">0</param>
-      <param name="limit_max">3.14159</param>
-      <param name="default">2.61799</param>
-      <command_interface name="position" />
-      <state_interface name="position" />
-    </joint>
-    <joint name="i02_leftHand_ThumbMid_joint">
-      <param name="virtual_pin">4</param>
-      <param name="servo_type">180</param>
-      <param name="offset">0</param>
-      <param name="direction">1</param>
-      <param name="scale">1</param>
-      <param name="limit_min">0</param>
-      <param name="limit_max">3.14159</param>
-      <param name="default">0</param>
-      <command_interface name="position" />
-      <state_interface name="position" />
-    </joint>
-    <joint name="i02_leftHand_indexPhal_joint">
-      <param name="virtual_pin">5</param>
-      <param name="servo_type">180</param>
-      <param name="offset">0</param>
-      <param name="direction">1</param>
-      <param name="scale">1</param>
-      <param name="limit_min">0</param>
-      <param name="limit_max">3.14159</param>
-      <param name="default">0</param>
-      <command_interface name="position" />
-      <state_interface name="position" />
-    </joint>
-    <joint name="i02_leftHand_majeurePhal_joint">
-      <param name="virtual_pin">6</param>
-      <param name="servo_type">180</param>
-      <param name="offset">0</param>
-      <param name="direction">1</param>
-      <param name="scale">1</param>
-      <param name="limit_min">0</param>
-      <param name="limit_max">3.14159</param>
-      <param name="default">0</param>
-      <command_interface name="position" />
-      <state_interface name="position" />
-    </joint>
-    <joint name="i02_leftHand_ringFingerPhal_joint">
-      <param name="virtual_pin">7</param>
-      <param name="servo_type">180</param>
-      <param name="offset">0</param>
-      <param name="direction">1</param>
-      <param name="scale">1</param>
-      <param name="limit_min">0</param>
-      <param name="limit_max">3.14159</param>
-      <param name="default">0</param>
-      <command_interface name="position" />
-      <state_interface name="position" />
-    </joint>
-    <joint name="i02_leftHand_pinkyPhal_joint">
-      <param name="virtual_pin">8</param>
-      <param name="servo_type">180</param>
-      <param name="offset">0</param>
-      <param name="direction">1</param>
-      <param name="scale">1</param>
-      <param name="limit_min">0</param>
-      <param name="limit_max">3.14159</param>
-      <param name="default">0</param>
-      <command_interface name="position" />
-      <state_interface name="position" />
-    </joint>
-    <joint name="right_shoulder_z_joint">
-      <param name="virtual_pin">9</param>
-      <param name="servo_type">180</param>
-      <param name="offset">1.5708</param>
-      <param name="direction">-1</param>
-      <param name="scale">1</param>
-      <param name="limit_min">0</param>
-      <param name="limit_max">3.14159</param>
-      <param name="default">1.5708</param>
-      <command_interface name="position" />
-      <state_interface name="position" />
-    </joint>
-    <joint name="right_shoulder_x_joint">
-      <param name="virtual_pin">10</param>
-      <param name="servo_type">180</param>
-      <param name="offset">0</param>
-      <param name="direction">1</param>
-      <param name="scale">1</param>
-      <param name="limit_min">0</param>
-      <param name="limit_max">3.14159</param>
-      <param name="default">0</param>
-      <command_interface name="position" />
-      <state_interface name="position" />
-    </joint>
-    <joint name="right_elbow_x_joint">
-      <param name="virtual_pin">11</param>
-      <param name="servo_type">180</param>
-      <param name="offset">0</param>
-      <param name="direction">1</param>
-      <param name="scale">1</param>
-      <param name="limit_min">0</param>
-      <param name="limit_max">3.14159</param>
-      <param name="default">0</param>
-      <command_interface name="position" />
-      <state_interface name="position" />
-    </joint>
-    <joint name="right_wrist_z_joint">
-      <param name="virtual_pin">12</param>
-      <param name="servo_type">180</param>
-      <param name="offset">2.61799</param>
-      <param name="direction">-1</param>
-      <param name="scale">1</param>
-      <param name="limit_min">0</param>
-      <param name="limit_max">3.14159</param>
-      <param name="default">2.61799</param>
-      <command_interface name="position" />
-      <state_interface name="position" />
-    </joint>
-    <joint name="i02_rightHand_ThumbMid_joint">
-      <param name="virtual_pin">13</param>
-      <param name="servo_type">180</param>
-      <param name="offset">0</param>
-      <param name="direction">1</param>
-      <param name="scale">1</param>
-      <param name="limit_min">0</param>
-      <param name="limit_max">3.14159</param>
-      <param name="default">0</param>
-      <command_interface name="position" />
-      <state_interface name="position" />
-    </joint>
-    <joint name="i02_rightHand_indexPhal_joint">
-      <param name="virtual_pin">14</param>
-      <param name="servo_type">180</param>
-      <param name="offset">0</param>
-      <param name="direction">1</param>
-      <param name="scale">1</param>
-      <param name="limit_min">0</param>
-      <param name="limit_max">3.14159</param>
-      <param name="default">0</param>
-      <command_interface name="position" />
-      <state_interface name="position" />
-    </joint>
-    <joint name="i02_rightHand_majeurePhal_joint">
-      <param name="virtual_pin">15</param>
-      <param name="servo_type">180</param>
-      <param name="offset">0</param>
-      <param name="direction">1</param>
-      <param name="scale">1</param>
-      <param name="limit_min">0</param>
-      <param name="limit_max">3.14159</param>
-      <param name="default">0</param>
-      <command_interface name="position" />
-      <state_interface name="position" />
-    </joint>
-    <joint name="i02_rightHand_ringFingerPhal_joint">
-      <param name="virtual_pin">16</param>
-      <param name="servo_type">180</param>
-      <param name="offset">0</param>
-      <param name="direction">1</param>
-      <param name="scale">1</param>
-      <param name="limit_min">0</param>
-      <param name="limit_max">3.14159</param>
-      <param name="default">0</param>
-      <command_interface name="position" />
-      <state_interface name="position" />
-    </joint>
-    <joint name="i02_rightHand_pinkyPhal_joint">
-      <param name="virtual_pin">17</param>
-      <param name="servo_type">180</param>
-      <param name="offset">0</param>
-      <param name="direction">1</param>
-      <param name="scale">1</param>
-      <param name="limit_min">0</param>
-      <param name="limit_max">3.14159</param>
-      <param name="default">0</param>
-      <command_interface name="position" />
-      <state_interface name="position" />
-    </joint>
-  </ros2_control>
-  <ros2_control name="LucyHardwareTorsoHead" type="system">
-    <hardware>
-      <plugin>gz_ros2_control/GazeboSimSystem</plugin>
-    </hardware>
-    <joint name="left_shoulder_y_joint">
-      <param name="virtual_pin">0</param>
-      <param name="servo_type">180</param>
-      <param name="offset">0</param>
-      <param name="direction">1</param>
-      <param name="scale">1</param>
-      <param name="limit_min">0</param>
-      <param name="limit_max">3.14159</param>
-      <param name="default">0</param>
-      <command_interface name="position" />
-      <state_interface name="position" />
-    </joint>
-    <joint name="right_shoulder_y_joint">
-      <param name="virtual_pin">1</param>
-      <param name="servo_type">180</param>
-      <param name="offset">0</param>
-      <param name="direction">1</param>
-      <param name="scale">1</param>
-      <param name="limit_min">0</param>
-      <param name="limit_max">3.14159</param>
-      <param name="default">0</param>
-      <command_interface name="position" />
-      <state_interface name="position" />
-    </joint>
-    <joint name="torso_z_joint">
-      <param name="virtual_pin">2</param>
-      <param name="servo_type">180</param>
-      <param name="offset">2.35619</param>
-      <param name="direction">1</param>
-      <param name="scale">1</param>
-      <param name="limit_min">0</param>
-      <param name="limit_max">3.14159</param>
-      <param name="default">2.35619</param>
-      <command_interface name="position" />
-      <state_interface name="position" />
-    </joint>
-    <joint name="torso_y_joint">
-      <param name="virtual_pin">3</param>
-      <param name="servo_type">180</param>
-      <param name="offset">1.5708</param>
-      <param name="direction">1</param>
-      <param name="scale">1</param>
-      <param name="limit_min">0</param>
-      <param name="limit_max">3.14159</param>
-      <param name="default">1.5708</param>
+      <param name="offset">0</param>
+      <param name="direction">1</param>
+      <param name="scale">1</param>
+      <param name="limit_min">0</param>
+      <param name="limit_max">3.14159</param>
+      <param name="default">0</param>
       <command_interface name="position" />
       <state_interface name="position" />
@@ -361,4 +140,225 @@
     <joint name="i02_head_left_eye_horizontal_joint">
       <param name="virtual_pin">11</param>
+      <param name="servo_type">180</param>
+      <param name="offset">1.5708</param>
+      <param name="direction">1</param>
+      <param name="scale">1</param>
+      <param name="limit_min">0</param>
+      <param name="limit_max">3.14159</param>
+      <param name="default">1.5708</param>
+      <command_interface name="position" />
+      <state_interface name="position" />
+    </joint>
+  </ros2_control>
+  <ros2_control name="LucyHardwareRight" type="system">
+    <hardware>
+      <plugin>gz_ros2_control/GazeboSimSystem</plugin>
+    </hardware>
+    <joint name="i02_leftHand_ThumbMid_joint">
+      <param name="virtual_pin">0</param>
+      <param name="servo_type">180</param>
+      <param name="offset">0</param>
+      <param name="direction">1</param>
+      <param name="scale">0.84082</param>
+      <param name="limit_min">0</param>
+      <param name="limit_max">1.39626</param>
+      <param name="default">0</param>
+      <command_interface name="position" />
+      <state_interface name="position" />
+    </joint>
+    <joint name="i02_leftHand_indexPhal_joint">
+      <param name="virtual_pin">1</param>
+      <param name="servo_type">180</param>
+      <param name="offset">0</param>
+      <param name="direction">1</param>
+      <param name="scale">1</param>
+      <param name="limit_min">0</param>
+      <param name="limit_max">3.14159</param>
+      <param name="default">0</param>
+      <command_interface name="position" />
+      <state_interface name="position" />
+    </joint>
+    <joint name="i02_leftHand_majeurePhal_joint">
+      <param name="virtual_pin">2</param>
+      <param name="servo_type">180</param>
+      <param name="offset">0</param>
+      <param name="direction">1</param>
+      <param name="scale">1</param>
+      <param name="limit_min">0</param>
+      <param name="limit_max">3.14159</param>
+      <param name="default">0</param>
+      <command_interface name="position" />
+      <state_interface name="position" />
+    </joint>
+    <joint name="i02_leftHand_ringFingerPhal_joint">
+      <param name="virtual_pin">3</param>
+      <param name="servo_type">180</param>
+      <param name="offset">0</param>
+      <param name="direction">1</param>
+      <param name="scale">1</param>
+      <param name="limit_min">0</param>
+      <param name="limit_max">3.14159</param>
+      <param name="default">0</param>
+      <command_interface name="position" />
+      <state_interface name="position" />
+    </joint>
+    <joint name="i02_leftHand_pinkyPhal_joint">
+      <param name="virtual_pin">4</param>
+      <param name="servo_type">180</param>
+      <param name="offset">0</param>
+      <param name="direction">1</param>
+      <param name="scale">1</param>
+      <param name="limit_min">0</param>
+      <param name="limit_max">3.14159</param>
+      <param name="default">0</param>
+      <command_interface name="position" />
+      <state_interface name="position" />
+    </joint>
+    <joint name="left_wrist_z_joint">
+      <param name="virtual_pin">5</param>
+      <param name="servo_type">180</param>
+      <param name="offset">2.61799</param>
+      <param name="direction">1</param>
+      <param name="scale">1</param>
+      <param name="limit_min">0</param>
+      <param name="limit_max">3.14159</param>
+      <param name="default">2.61799</param>
+      <command_interface name="position" />
+      <state_interface name="position" />
+    </joint>
+    <joint name="i02_rightHand_ThumbMid_joint">
+      <param name="virtual_pin">6</param>
+      <param name="servo_type">180</param>
+      <param name="offset">0</param>
+      <param name="direction">1</param>
+      <param name="scale">0.82291</param>
+      <param name="limit_min">0</param>
+      <param name="limit_max">1.39626</param>
+      <param name="default">0</param>
+      <command_interface name="position" />
+      <state_interface name="position" />
+    </joint>
+    <joint name="i02_rightHand_indexPhal_joint">
+      <param name="virtual_pin">7</param>
+      <param name="servo_type">180</param>
+      <param name="offset">0</param>
+      <param name="direction">1</param>
+      <param name="scale">1</param>
+      <param name="limit_min">0</param>
+      <param name="limit_max">3.14159</param>
+      <param name="default">0.017453292519943295</param>
+      <command_interface name="position" />
+      <state_interface name="position" />
+    </joint>
+    <joint name="i02_rightHand_majeurePhal_joint">
+      <param name="virtual_pin">8</param>
+      <param name="servo_type">180</param>
+      <param name="offset">0</param>
+      <param name="direction">1</param>
+      <param name="scale">1</param>
+      <param name="limit_min">0</param>
+      <param name="limit_max">3.14159</param>
+      <param name="default">0</param>
+      <command_interface name="position" />
+      <state_interface name="position" />
+    </joint>
+    <joint name="i02_rightHand_ringFingerPhal_joint">
+      <param name="virtual_pin">9</param>
+      <param name="servo_type">180</param>
+      <param name="offset">0</param>
+      <param name="direction">1</param>
+      <param name="scale">1</param>
+      <param name="limit_min">0</param>
+      <param name="limit_max">3.14159</param>
+      <param name="default">0</param>
+      <command_interface name="position" />
+      <state_interface name="position" />
+    </joint>
+    <joint name="i02_rightHand_pinkyPhal_joint">
+      <param name="virtual_pin">10</param>
+      <param name="servo_type">180</param>
+      <param name="offset">0</param>
+      <param name="direction">1</param>
+      <param name="scale">1</param>
+      <param name="limit_min">0</param>
+      <param name="limit_max">3.14159</param>
+      <param name="default">0</param>
+      <command_interface name="position" />
+      <state_interface name="position" />
+    </joint>
+    <joint name="right_wrist_z_joint">
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